File: kicad-scyboard/scyboard.kicad_pcb (KiCad board)
At the start: 2 copper layers, 144 x 96.5 mm, 92 parts

Commit message: Update KiCad
Parts:
- moved PWR1 0.16 mm to (168.1, 92.9)
Routing:
- net C2: track 9.64 -> 240.1 mm, vias 0 -> 4
- net C0: track 9.64 -> 203.6 mm, vias 0 -> 5
- net C1: track 9.64 -> 203.0 mm, vias 0 -> 6
- net C4: track 9.64 -> 177.1 mm, vias 0 -> 4
- net C3: track 9.64 -> 176.5 mm, vias 0 -> 4
- net R0: track 9.63 -> 175.7 mm, vias 0 -> 7
- net R3: track 9.63 -> 173.7 mm, vias 0 -> 3
- net R2: track 9.63 -> 172.6 mm, vias 0 -> 6
- net R1: track 9.63 -> 166.9 mm, vias 0 -> 8
- net C5: track 9.64 -> 153.0 mm, vias 0 -> 3
- net RAW: track 9.64 -> 114.4 mm, vias 0 -> 3
- net GND: track 28.9 -> 108.1 mm, vias 0 -> 2
- net RST: track 9.64 -> 51.5 mm, vias 0 -> 1
- net BAT_P: track 0.00 -> 18.6 mm, vias 0 -> 1
- net space_cluster_F: track 0.00 -> 14.5 mm
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
Commit message: Compile
Parts:
- removed D23, D24, D25, D26, D27, D28, D29, D30, D31, D32, D33, D34, D35, D36, D37, D38, D39, D40, D41, D42, D43, D44: , ceoloide:diode_tht_sod123
- removed S23, S24, S25, S26, S27, S28, S29, S30, S31, S32, S33, S34, S35, S36, S37, S38, S39, S40, S41, S42, S43, S44: , ceoloide:switch_choc_v1_v2
- moved PWR1 0.16 mm to (168.2, 92.9)
Connections:
- JST1 pad 1: BAT_P -> GND
- JST1 pad 2: GND -> BAT_P
- MCU1 pad 1: MCU1_1 -> RAW
- MCU1 pad 10: MCU1_10 -> C5
- MCU1 pad 11: MCU1_11 -> P16
- MCU1 pad 12: MCU1_12 -> P10
- MCU1 pad 13: MCU1_13 -> P9
- MCU1 pad 14: MCU1_14 -> R3
- MCU1 pad 15: MCU1_15 -> R2
- MCU1 pad 16: MCU1_16 -> R1
- MCU1 pad 17: MCU1_17 -> R0
- MCU1 pad 18: MCU1_18 -> CS
- MCU1 pad 19: MCU1_19 -> SCL
- MCU1 pad 2: MCU1_2 -> GND
- MCU1 pad 20: MCU1_20 -> SDA
- MCU1 pad 21: MCU1_21 -> GND
- MCU1 pad 22: MCU1_22 -> GND
- MCU1 pad 23: MCU1_23 -> DAT
- MCU1 pad 24: MCU1_24 -> LED
- MCU1 pad 3: MCU1_3 -> RST
- MCU1 pad 4: MCU1_4 -> VCC
- MCU1 pad 5: MCU1_5 -> C0
- MCU1 pad 6: MCU1_6 -> C1
- MCU1 pad 7: MCU1_7 -> C2
- MCU1 pad 8: MCU1_8 -> C3
- MCU1 pad 9: MCU1_9 -> C4
- PWR1 pad 1: BAT_P -> (no net)
Routing:
- net C2: track 240.1 -> 0.00 mm, vias 4 -> 0
- net C0: track 203.6 -> 0.00 mm, vias 5 -> 0
- net C1: track 203.0 -> 0.00 mm, vias 6 -> 0
- net C4: track 177.1 -> 0.00 mm, vias 4 -> 0
- net C3: track 176.5 -> 0.00 mm, vias 4 -> 0
- net R0: track 175.7 -> 0.00 mm, vias 7 -> 0
- net R3: track 173.7 -> 0.00 mm, vias 3 -> 0
- net R2: track 172.6 -> 0.00 mm, vias 6 -> 0
- net R1: track 166.9 -> 0.00 mm, vias 8 -> 0
- net C5: track 153.0 -> 0.00 mm, vias 3 -> 0
- net RAW: track 114.4 -> 0.00 mm, vias 3 -> 0
- net GND: track 108.1 -> 0.00 mm, vias 2 -> 0
- net RST: track 51.5 -> 0.00 mm, vias 1 -> 0
- net BAT_P: track 18.6 -> 0.00 mm, vias 1 -> 0
- net space_cluster_F: track 14.5 -> 0.00 mm
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