File: kicad-scyboard/scyboard.kicad_pcb (KiCad board)
At the start: 2 copper layers, 144 x 96.5 mm, 48 parts

Commit message: Compile
Parts:
- added G***: LOGO, custom:scyboard_logo, F.Cu at (91.3, 103.3)
Other:
- board text added: "RESET"
- board text added: "scyboard https://github.com/Scybin/scyboard"

Commit message: Compile
Parts:
- moved JST1 1.90 mm to (163.8, 89.0)
- moved G*** 0.22 mm to (91.2, 103.2)
- moved PWR1 0.20 mm to (168.2, 92.9)
Connections:
- MCU1 pad 1: RAW -> LED
- MCU1 pad 10: C5 -> R2
- MCU1 pad 11: P16 -> R3
- MCU1 pad 12: P10 -> P9
- MCU1 pad 13: P9 -> P10
- MCU1 pad 14: R3 -> P16
- MCU1 pad 15: R2 -> C5
- MCU1 pad 16: R1 -> C4
- MCU1 pad 17: R0 -> C3
- MCU1 pad 18: CS -> C2
- MCU1 pad 19: SCL -> C1
- MCU1 pad 2: GND -> DAT
- MCU1 pad 20: SDA -> C0
- MCU1 pad 21: GND -> VCC
- MCU1 pad 22: GND -> RST
- MCU1 pad 23: DAT -> GND
- MCU1 pad 24: LED -> RAW
- MCU1 pad 3: RST -> GND
- MCU1 pad 4: VCC -> GND
- MCU1 pad 5: C0 -> SDA
- MCU1 pad 6: C1 -> SCL
- MCU1 pad 7: C2 -> CS
- MCU1 pad 8: C3 -> R0
- MCU1 pad 9: C4 -> R1
Routing:
- net R2: track 207.8 -> 157.7 mm, vias 3 -> 7
- net R0: track 129.9 -> 158.1 mm, vias 0 -> 1
- net C4: track 105.1 -> 77.0 mm, vias 1 -> 0
- net C0: track 160.0 -> 139.6 mm
- net RST: track 34.8 -> 48.1 mm
- net C1: track 135.4 -> 122.8 mm
- net C2: track 153.3 -> 141.4 mm, vias 1 -> 3
- net C3: track 139.9 -> 128.5 mm, vias 3 -> 2
- net R1: track 162.9 -> 172.9 mm, vias 4 -> 6
- net C5: track 90.6 -> 81.6 mm, vias 1 -> 0
- net RAW: track 45.8 -> 51.9 mm
- net GND: track 67.8 -> 64.0 mm
- net BAT_P: track 4.61 -> 3.00 mm
- net R3: track 111.3 -> 112.4 mm, vias 2 -> 3
Other:
- board text added: "BATTERY"

Commit message: Compile
Parts:
- removed G***: LOGO, custom:scyboard_logo
- added MH1: , ceoloide:mounting_hole_npth, F.Cu at (59.5, 72.7)
- added MH2: , ceoloide:mounting_hole_npth, F.Cu at (59.5, 89.7)
- added MH3: , ceoloide:mounting_hole_npth, F.Cu at (108.5, 92.6)
- added MH4: , ceoloide:mounting_hole_npth, F.Cu at (95.5, 56.3)
- added MH5: , ceoloide:mounting_hole_npth, F.Cu at (131.5, 63.5)
- added MH6: , ceoloide:mounting_hole_npth, F.Cu at (163.7, 108.5)
- turned RST1 to 0 degrees
- turned JST1 to 90 degrees
Routing:
- net R1: track 172.9 -> 0.00 mm, vias 6 -> 0
- net R0: track 158.1 -> 0.00 mm, vias 1 -> 0
- net R2: track 157.7 -> 0.00 mm, vias 7 -> 0
- net C2: track 141.4 -> 0.00 mm, vias 3 -> 0
- net C0: track 139.6 -> 0.00 mm, vias 1 -> 0
- net C3: track 128.5 -> 0.00 mm, vias 2 -> 0
- net C1: track 122.8 -> 0.00 mm, vias 1 -> 0
- net R3: track 112.4 -> 0.00 mm, vias 3 -> 0
- net C5: track 81.6 -> 0.00 mm
- net C4: track 77.0 -> 0.00 mm
- net GND: track 64.0 -> 0.00 mm
- net RAW: track 51.9 -> 0.00 mm, vias 1 -> 0
- net RST: track 48.1 -> 0.00 mm, vias 1 -> 0
- net space_cluster_B: track 3.89 -> 0.00 mm
- net layer_cluster_B: track 3.85 -> 0.00 mm
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Other:
- board size 144 x 96.5 mm -> 143.9 x 96.5 mm
- board text removed: "BATTERY"
- board text removed: "RESET"
- board text removed: "scyboard https://github.com/Scybin/scyboard"

Commit message: Compile
Parts:
- added REF**: custom_case, custom:custom_case, F.Cu at (100.1, 69.5)
- S1, S10, S11, S12, S13, S14, S15, S16, S17, S18, S19, S2, S20, S22, S3, S4, S5, S6, S7, S8, S9: footprint ceoloide:switch_choc_v1_v2 -> custom:custom_switch_choc_v1
- S21: footprint ceoloide:switch_choc_v1_v2 -> custom:custom_switch_choc_v1_1.5u
- turned RST1 to -90 degrees
- turned JST1 to -90 degrees
Other:
- board size 143.9 x 96.5 mm -> 144 x 96.5 mm

Commit message: Compile
Parts:
- removed REF**: custom_case, custom:custom_case
- added D23: , ceoloide:diode_tht_sod123, F.Cu at (57.8, 98.5)
- added D24: , ceoloide:diode_tht_sod123, F.Cu at (57.8, 81.5)
- added D25: , ceoloide:diode_tht_sod123, F.Cu at (57.8, 64.5)
- added D26: , ceoloide:diode_tht_sod123, F.Cu at (75.8, 96.7)
- added D27: , ceoloide:diode_tht_sod123, F.Cu at (75.8, 79.7)
- added D28: , ceoloide:diode_tht_sod123, F.Cu at (75.8, 62.7)
- added D29: , ceoloide:diode_tht_sod123, F.Cu at (93.8, 84.8)
- added D30: , ceoloide:diode_tht_sod123, F.Cu at (93.8, 67.8)
- added D31: , ceoloide:diode_tht_sod123, F.Cu at (93.8, 50.8)
- added D32: , ceoloide:diode_tht_sod123, F.Cu at (111.8, 80.3)
- added D33: , ceoloide:diode_tht_sod123, F.Cu at (111.8, 63.3)
- added D34: , ceoloide:diode_tht_sod123, F.Cu at (111.8, 46.3)
- added D35: , ceoloide:diode_tht_sod123, F.Cu at (129.8, 84.8)
- added D36: , ceoloide:diode_tht_sod123, F.Cu at (129.8, 67.8)
- added D37: , ceoloide:diode_tht_sod123, F.Cu at (129.8, 50.8)
- added D38: , ceoloide:diode_tht_sod123, F.Cu at (147.8, 87.5)
- added D39: , ceoloide:diode_tht_sod123, F.Cu at (147.8, 70.5)
- added D40: , ceoloide:diode_tht_sod123, F.Cu at (147.8, 53.5)
- added D41: , ceoloide:diode_tht_sod123, F.Cu at (120.8, 101.8)
- added D42: , ceoloide:diode_tht_sod123, F.Cu at (140.3, 106.8)
- added D43: , ceoloide:diode_tht_sod123, F.Cu at (150.4, 116.1)
- added D44: , ceoloide:diode_tht_sod123, F.Cu at (165.7, 125.6)
- S1, S10, S11, S12, S13, S14, S15, S16, S17, S18, S19, S2, S20, S22, S3, S4, S5, S6, S7, S8, S9: footprint custom:custom_switch_choc_v1 -> ceoloide:switch_choc_v1_v2
- S21: footprint custom:custom_switch_choc_v1_1.5u -> ceoloide:switch_choc_v1_v2
- moved MH6 57.4 mm to (108.5, 92.6)
- moved MH5 55.3 mm to (163.7, 108.5)
- moved MH3 44.4 mm to (77.5, 60.8)
- moved MH4 36.7 mm to (131.5, 63.5)
- moved MH1 2.06 mm to (58.5, 74.5)
- moved MH2 2.06 mm to (58.5, 91.5)
Connections:
- JST1 pad 1: GND -> BAT_P
- JST1 pad 2: BAT_P -> GND
- MCU1 pad 1: LED -> MCU1_1
- MCU1 pad 10: R2 -> MCU1_10
- MCU1 pad 11: R3 -> MCU1_11
- MCU1 pad 12: P9 -> MCU1_12
- MCU1 pad 13: P10 -> MCU1_13
- MCU1 pad 14: P16 -> MCU1_14
- MCU1 pad 15: C5 -> MCU1_15
- MCU1 pad 16: C4 -> MCU1_16
- MCU1 pad 17: C3 -> MCU1_17
- MCU1 pad 18: C2 -> MCU1_18
- MCU1 pad 19: C1 -> MCU1_19
- MCU1 pad 2: DAT -> MCU1_2
- MCU1 pad 20: C0 -> MCU1_20
- MCU1 pad 21: VCC -> MCU1_21
- MCU1 pad 22: RST -> MCU1_22
- MCU1 pad 23: GND -> MCU1_23
- MCU1 pad 24: RAW -> MCU1_24
- MCU1 pad 3: GND -> MCU1_3
- MCU1 pad 4: GND -> MCU1_4
- MCU1 pad 5: SDA -> MCU1_5
- MCU1 pad 6: SCL -> MCU1_6
- MCU1 pad 7: CS -> MCU1_7
- MCU1 pad 8: R0 -> MCU1_8
- MCU1 pad 9: R1 -> MCU1_9
- PWR1 pad 1: (no net) -> BAT_P
Routing:
- net C0: track 0.00 -> 195.6 mm, vias 0 -> 4
- net C2: track 0.00 -> 191.2 mm, vias 0 -> 5
- net C3: track 0.00 -> 171.3 mm, vias 0 -> 5
- net R2: track 0.00 -> 170.3 mm, vias 0 -> 7
- net R0: track 0.00 -> 166.9 mm, vias 0 -> 8
- net R3: track 0.00 -> 162.5 mm, vias 0 -> 6
- net R1: track 0.00 -> 159.2 mm, vias 0 -> 7
- net C4: track 0.00 -> 149.0 mm, vias 0 -> 6
- net C5: track 0.00 -> 146.9 mm, vias 0 -> 6
- net GND: track 0.00 -> 91.1 mm, vias 0 -> 4
- net C1: track 0.00 -> 66.8 mm, vias 0 -> 3
- net RAW: track 0.00 -> 64.0 mm, vias 0 -> 1
- net RST: track 0.00 -> 57.2 mm, vias 0 -> 2
- net space_cluster_B: track 0.00 -> 25.5 mm, vias 0 -> 1
- net layer_cluster_B: track 0.00 -> 25.5 mm, vias 0 -> 1
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
Commit message: Compile
Parts:
- moved MH3 8.86 mm to (75.0, 52.3)
- turned JST1 to 90 degrees
- turned RST1 to 0 degrees
Routing:
- net C0: track 195.6 -> 34.6 mm, vias 4 -> 3
- net R2: track 170.3 -> 9.84 mm, vias 7 -> 0
- net R0: track 166.9 -> 9.84 mm, vias 8 -> 0
- net R3: track 162.5 -> 9.84 mm, vias 6 -> 0
- net R1: track 159.2 -> 9.84 mm, vias 7 -> 0
- net C2: track 191.2 -> 42.9 mm, vias 5 -> 4
- net C3: track 171.3 -> 42.9 mm, vias 5 -> 4
- net C4: track 149.0 -> 42.9 mm, vias 6 -> 4
- net C5: track 146.9 -> 42.9 mm, vias 6 -> 4
- net GND: track 91.1 -> 29.5 mm, vias 4 -> 0
- net RAW: track 64.0 -> 9.83 mm, vias 1 -> 0
- net RST: track 57.2 -> 9.83 mm, vias 2 -> 0
- net C1: track 66.8 -> 34.6 mm
- net BAT_P: track 18.2 -> 0.00 mm, vias 2 -> 0
- net space_cluster_B: track 25.5 -> 19.1 mm
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
Commit message: Compile
Parts:
- moved PWR1 0.19 mm to (168.1, 92.9)
Routing:
- net (no net): track 0.00 -> 337.7 mm
- net GND: track 29.5 -> 0.00 mm
- net P9: track 9.84 -> 0.00 mm
- net DAT: track 9.84 -> 0.00 mm
- net R2: track 9.84 -> 0.00 mm
- net LED: track 9.84 -> 0.00 mm
- net CS: track 9.84 -> 0.00 mm
- net SCL: track 9.84 -> 0.00 mm
- net SDA: track 9.84 -> 0.00 mm
- net R3: track 9.84 -> 0.00 mm
- net R1: track 9.84 -> 0.00 mm
- net R0: track 9.84 -> 0.00 mm
- net C4: track 42.9 -> 33.1 mm
- net C5: track 42.9 -> 33.1 mm
- net RAW: track 9.83 -> 0.00 mm
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Other:
- board size 144 x 96.5 mm -> 143.9 x 96.5 mm

Commit message: Compile
Parts:
- moved JST1 0.62 mm to (163.2, 89.0), turned to -90 degrees
- moved PWR1 0.33 mm to (167.7, 92.9)
- turned RST1 to -90 degrees
Routing:
- net (no net): track 337.7 -> 0.00 mm
- net C0: track 24.8 -> 207.9 mm, vias 3 -> 4
- net R0: track 0.00 -> 182.8 mm, vias 0 -> 7
- net R2: track 0.00 -> 174.8 mm, vias 0 -> 7
- net R3: track 0.00 -> 164.1 mm, vias 0 -> 5
- net R1: track 0.00 -> 161.6 mm, vias 0 -> 8
- net C2: track 33.1 -> 188.3 mm, vias 4 -> 5
- net C3: track 33.1 -> 177.8 mm, vias 4 -> 5
- net C1: track 24.8 -> 161.6 mm, vias 3 -> 4
- net C4: track 33.1 -> 156.5 mm
- net C5: track 33.1 -> 135.1 mm, vias 4 -> 5
- net GND: track 0.00 -> 98.2 mm, vias 0 -> 3
- net RAW: track 0.00 -> 67.0 mm, vias 0 -> 1
- net RST: track 0.00 -> 55.4 mm, vias 0 -> 1
- net BAT_P: track 0.00 -> 19.2 mm, vias 0 -> 1
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Other:
- board size 143.9 x 96.5 mm -> 148.5 x 100.9 mm
