File: ergogen/output/pcbs/scyboard.kicad_pcb (KiCad board)
At the start: 2 copper layers, 143.9 x 96.5 mm, 50 parts

Commit message: Compile
Parts:
- added MH3: , ceoloide:mounting_hole_npth, F.Cu at (59.0, 108.5)
Changed lines of the file:
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@@
+    )
+  )
+  (footprint "ceoloide:mounting_hole_npth"
+    (layer "F.Cu")
+    (at 59 108.5 0)
+    (property "Reference" "MH3"
+      (at 0 2.55 0)
+      (layer "F.SilkS")
+      hide
+      (effects (font (size 1 1) (thickness 0.15)))
+    )
+    (pad "" np_thru_hole circle
+      (at 0 0 0)
+      (size 4.3 4.3)
+      (drill 4.3)
+      (layers "*.Cu" "*.Mask")
     )
   )

Commit message: Compile
Parts:
- moved MH3 63.1 mm to (122.0, 111.8)
Changed lines of the file:
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@@
   (footprint "ceoloide:mounting_hole_npth"
     (layer "F.Cu")
-    (at 59 108.5 0)
+    (at 122 111.82 0)
     (property "Reference" "MH3"
       (at 0 2.55 0)

Commit message: Compile
Parts:
- moved MH3 26.2 mm to (99.5, 98.3)
Changed lines of the file:
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@@
   (footprint "ceoloide:mounting_hole_npth"
     (layer "F.Cu")
-    (at 122 111.82 0)
+    (at 99.5 98.32 0)
     (property "Reference" "MH3"
       (at 0 2.55 0)

Commit message: Compile
Parts:
- moved MH3 10.7 mm to (108.5, 92.6)
Changed lines of the file:
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@@
   (footprint "ceoloide:mounting_hole_npth"
     (layer "F.Cu")
-    (at 99.5 98.32 0)
+    (at 108.5 92.57 0)
     (property "Reference" "MH3"
       (at 0 2.55 0)

Commit message: Compile
Parts:
- added MH4: , ceoloide:mounting_hole_npth, F.Cu at (131.0, 60.8)
- added MH5: , ceoloide:mounting_hole_npth, F.Cu at (130.1, 60.8)
Changed lines of the file:
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@@
+    )
+  )
+  (footprint "ceoloide:mounting_hole_npth"
+    (layer "F.Cu")
+    (at 131 60.81999999999999 0)
+    (property "Reference" "MH4"
+      (at 0 2.55 0)
+      (layer "F.SilkS")
+      hide
+      (effects (font (size 1 1) (thickness 0.15)))
+    )
+    (pad "" np_thru_hole circle
+      (at 0 0 0)
+      (size 4.3 4.3)
+      (drill 4.3)
+      (layers "*.Cu" "*.Mask")
+    )
+  )
+  (footprint "ceoloide:mounting_hole_npth"
+    (layer "F.Cu")
+    (at 130.1 60.81999999999999 0)
+    (property "Reference" "MH5"
+      (at 0 2.55 0)
+      (layer "F.SilkS")
+      hide
+      (effects (font (size 1 1) (thickness 0.15)))
+    )
+    (pad "" np_thru_hole circle
+      (at 0 0 0)
+      (size 4.3 4.3)
+      (drill 4.3)
+      (layers "*.Cu" "*.Mask")
     )
   )

Commit message: Compile
Parts:
- moved MH5 16.7 mm to (142.7, 71.8)
Changed lines of the file:
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@@
   (footprint "ceoloide:mounting_hole_npth"
     (layer "F.Cu")
-    (at 130.1 60.81999999999999 0)
+    (at 142.7 71.82 0)
     (property "Reference" "MH5"
       (at 0 2.55 0)

Commit message: Compile
Parts:
- moved MH5 40.9 mm to (160.7, 108.5)
- moved MH4 1.35 mm to (131.0, 62.2)
Changed lines of the file:
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@@
   (footprint "ceoloide:mounting_hole_npth"
     (layer "F.Cu")
-    (at 131 60.81999999999999 0)
+    (at 131 62.169999999999995 0)
     (property "Reference" "MH4"
       (at 0 2.55 0)
@@
   (footprint "ceoloide:mounting_hole_npth"
     (layer "F.Cu")
-    (at 142.7 71.82 0)
+    (at 160.7 108.52 0)
     (property "Reference" "MH5"
       (at 0 2.55 0)

Commit message: Compile
Parts:
- moved MH4 25.7 mm to (148.5, 81.0)
Changed lines of the file:
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@@
   (footprint "ceoloide:mounting_hole_npth"
     (layer "F.Cu")
-    (at 131 62.169999999999995 0)
+    (at 148.5 81.02 0)
     (property "Reference" "MH4"
       (at 0 2.55 0)
