File: ergogen/output/pcbs/scyboard.kicad_pcb (KiCad board)
At the start: 2 copper layers, 143.9 x 96.5 mm, 76 parts

Commit message: Compile
Parts:
- moved MH3 0.50 mm to (75.0, 52.3)
Changed lines of the file:
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@@
   (footprint "ceoloide:mounting_hole_npth"
     (layer "F.Cu")
-    (at 75.5 52.31999999999999 0)
+    (at 75 52.31999999999999 0)
     (property "Reference" "MH3"
       (at 0 2.55 0)

Commit message: Compile
Parts:
- moved PWR1 0.91 mm to (167.3, 92.9)
Changed lines of the file:
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@@
   (footprint "ceoloide:power_switch_smd_side"
     (layer "F.Cu")
-    (at 168.25 92.87 0)
+    (at 167.335 92.87 0)
     (property "Reference" "PWR1"
       (at -3.6 0 -90)

Commit message: Compile
Parts:
- moved PWR1 0.66 mm to (168.0, 92.9)
Changed lines of the file:
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@@
   (footprint "ceoloide:power_switch_smd_side"
     (layer "F.Cu")
-    (at 167.335 92.87 0)
+    (at 168 92.87 0)
     (property "Reference" "PWR1"
       (at -3.6 0 -90)

Commit message: Compile
Parts:
- moved JST1 4.21 mm to (159.6, 89.0)
- moved PWR1 0.06 mm to (168.1, 92.9)
Changed lines of the file:
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@@
   (footprint "ceoloide:power_switch_smd_side"
     (layer "F.Cu")
-    (at 168 92.87 0)
+    (at 168.055 92.87 0)
     (property "Reference" "PWR1"
       (at -3.6 0 -90)
@@
     (footprint "ceoloide:battery_connector_jst_ph_2"
         (layer "F.Cu")
-        (at 163.85 89.03 90)
+        (at 159.64 89.03 90)
         (property "Reference" "JST1"
             (at 0 4.8 90)
@@
         )
     )
-    (segment (start 165.65 90.03) (end 163.85 90.03) (width 0.25) (layer "F.Cu") (net 75))
-    (segment (start 165.65 90.03) (end 163.85 90.03) (width 0.25) (layer "B.Cu") (net 75))
-    (segment (start 165.65 88.03) (end 163.85 88.03) (width 0.25) (layer "F.Cu") (net 76))
-    (segment (start 165.65 88.03) (end 163.85 88.03) (width 0.25) (layer "B.Cu") (net 76))
+    (segment (start 161.44 90.03) (end 159.64 90.03) (width 0.25) (layer "F.Cu") (net 75))
+    (segment (start 161.44 90.03) (end 159.64 90.03) (width 0.25) (layer "B.Cu") (net 75))
+    (segment (start 161.44 88.03) (end 159.64 88.03) (width 0.25) (layer "F.Cu") (net 76))
+    (segment (start 161.44 88.03) (end 159.64 88.03) (width 0.25) (layer "B.Cu") (net 76))
   (footprint "ceoloide:mounting_hole_npth"
     (layer "F.Cu")

Commit message: Compile
Parts:
- moved JST1 4.21 mm to (163.8, 89.0)
Changed lines of the file:
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@@
     (footprint "ceoloide:battery_connector_jst_ph_2"
         (layer "F.Cu")
-        (at 159.64 89.03 90)
+        (at 163.845 89.03 90)
         (property "Reference" "JST1"
             (at 0 4.8 90)
@@
         )
     )
-    (segment (start 161.44 90.03) (end 159.64 90.03) (width 0.25) (layer "F.Cu") (net 75))
-    (segment (start 161.44 90.03) (end 159.64 90.03) (width 0.25) (layer "B.Cu") (net 75))
-    (segment (start 161.44 88.03) (end 159.64 88.03) (width 0.25) (layer "F.Cu") (net 76))
-    (segment (start 161.44 88.03) (end 159.64 88.03) (width 0.25) (layer "B.Cu") (net 76))
+    (segment (start 165.645 90.03) (end 163.845 90.03) (width 0.25) (layer "F.Cu") (net 75))
+    (segment (start 165.645 90.03) (end 163.845 90.03) (width 0.25) (layer "B.Cu") (net 75))
+    (segment (start 165.645 88.03) (end 163.845 88.03) (width 0.25) (layer "F.Cu") (net 76))
+    (segment (start 165.645 88.03) (end 163.845 88.03) (width 0.25) (layer "B.Cu") (net 76))
   (footprint "ceoloide:mounting_hole_npth"
     (layer "F.Cu")

Commit message: Compile
Parts:
- moved JST1 0.29 mm to (163.6, 89.0)
Changed lines of the file:
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@@
     (footprint "ceoloide:battery_connector_jst_ph_2"
         (layer "F.Cu")
-        (at 163.845 89.03 90)
+        (at 163.555 89.03 90)
         (property "Reference" "JST1"
             (at 0 4.8 90)
@@
         )
     )
-    (segment (start 165.645 90.03) (end 163.845 90.03) (width 0.25) (layer "F.Cu") (net 75))
-    (segment (start 165.645 90.03) (end 163.845 90.03) (width 0.25) (layer "B.Cu") (net 75))
-    (segment (start 165.645 88.03) (end 163.845 88.03) (width 0.25) (layer "F.Cu") (net 76))
-    (segment (start 165.645 88.03) (end 163.845 88.03) (width 0.25) (layer "B.Cu") (net 76))
+    (segment (start 165.35500000000002 90.03) (end 163.555 90.03) (width 0.25) (layer "F.Cu") (net 75))
+    (segment (start 165.35500000000002 90.03) (end 163.555 90.03) (width 0.25) (layer "B.Cu") (net 75))
+    (segment (start 165.35500000000002 88.03) (end 163.555 88.03) (width 0.25) (layer "F.Cu") (net 76))
+    (segment (start 165.35500000000002 88.03) (end 163.555 88.03) (width 0.25) (layer "B.Cu") (net 76))
   (footprint "ceoloide:mounting_hole_npth"
     (layer "F.Cu")

Commit message: Compile
Parts:
- moved JST1 0.33 mm to (163.9, 89.0)
- moved PWR1 0.33 mm to (168.4, 92.9)
Other:
- board size 143.9 x 96.5 mm -> 148.5 x 100.9 mm

Commit message: Compile
Parts:
- moved JST1 0.66 mm to (163.2, 89.0)
- moved PWR1 0.66 mm to (167.7, 92.9)
Changed lines of the file:
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@@
   (footprint "ceoloide:power_switch_smd_side"
     (layer "F.Cu")
-    (at 168.385 92.87 0)
+    (at 167.725 92.87 0)
     (property "Reference" "PWR1"
       (at -3.6 0 -90)
@@
     (footprint "ceoloide:battery_connector_jst_ph_2"
         (layer "F.Cu")
-        (at 163.885 89.03 90)
+        (at 163.225 89.03 90)
         (property "Reference" "JST1"
             (at 0 4.8 90)
@@
         )
     )
-    (segment (start 165.685 90.03) (end 163.885 90.03) (width 0.25) (layer "F.Cu") (net 75))
-    (segment (start 165.685 90.03) (end 163.885 90.03) (width 0.25) (layer "B.Cu") (net 75))
-    (segment (start 165.685 88.03) (end 163.885 88.03) (width 0.25) (layer "F.Cu") (net 76))
-    (segment (start 165.685 88.03) (end 163.885 88.03) (width 0.25) (layer "B.Cu") (net 76))
+    (segment (start 165.025 90.03) (end 163.225 90.03) (width 0.25) (layer "F.Cu") (net 75))
+    (segment (start 165.025 90.03) (end 163.225 90.03) (width 0.25) (layer "B.Cu") (net 75))
+    (segment (start 165.025 88.03) (end 163.225 88.03) (width 0.25) (layer "F.Cu") (net 76))
+    (segment (start 165.025 88.03) (end 163.225 88.03) (width 0.25) (layer "B.Cu") (net 76))
   (footprint "ceoloide:mounting_hole_npth"
     (layer "F.Cu")
