File: kicad/scyboard.kicad_pcb (KiCad board)
At the start: 2 copper layers, 148.5 x 100.9 mm, 77 parts

Commit message: Update PCB
Parts:
- removed G***: LOGO, custom:scyboard_logo
- added LOGO1: , custom:scyboard_logo, F.Cu at (91.0, 105.0)
Connections:
- net DAT renamed P0
- net LED renamed P1
- net SCL renamed P3
- net SDA renamed P2
- MCU1 pad 107: CS -> R0
- MCU1 pad 108: R0 -> R1
- MCU1 pad 109: R1 -> R2
- MCU1 pad 110: R2 -> R3
- MCU1 pad 111: R3 -> P8
Routing:
- net C0: track 200.5 -> 180.8 mm, vias 4 -> 3
- net C3: track 167.2 -> 183.5 mm, vias 5 -> 6
- net R0: track 170.6 -> 184.6 mm, vias 6 -> 9
- net R1: track 156.0 -> 167.6 mm, vias 9 -> 8
- net C4: track 158.3 -> 147.5 mm, vias 5 -> 6
- net P8: track 0.00 -> 9.96 mm
- net CS: track 9.96 -> 0.00 mm
- net C5: track 143.6 -> 134.7 mm, vias 6 -> 4
- net RAW: track 72.2 -> 79.8 mm
- net C1: track 166.1 -> 160.6 mm
- net R2: track 178.6 -> 173.5 mm, vias 7 -> 8
- net R3: track 161.3 -> 165.5 mm
- net BAT_P: track 13.7 -> 16.3 mm, vias 2 -> 1
- net RST: track 51.3 -> 48.9 mm, vias 1 -> 2
- net C2: track 182.9 -> 181.2 mm
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- added copper zone on B.Cu, net (none)
- added copper zone on F.Cu, net (none)
- removed copper zone on B.Cu, net C0
- removed copper zone on F.Cu, net C0

Commit message: Generate gerbers
Parts:
- moved MH4 27.4 mm to (115.6, 41.2)
- moved MH2 27.1 mm to (79.8, 108.2)
- moved MH5 21.5 mm to (152.2, 90.3)
- moved MH3 20.6 mm to (92.4, 41.2)
- moved MH1 19.5 mm to (57.8, 55.0)
Routing:
- net C3: track 183.5 -> 170.8 mm, vias 6 -> 5
- net C4: track 147.5 -> 159.8 mm, vias 6 -> 4
- net R0: track 184.6 -> 173.4 mm, vias 9 -> 8
- net C1: track 160.6 -> 169.8 mm
- net R2: track 173.5 -> 165.2 mm
- net C2: track 181.2 -> 174.0 mm, vias 5 -> 6
- net R1: track 167.6 -> 173.7 mm, vias 8 -> 7
- net C0: track 180.8 -> 185.4 mm
- net GND: track 106.4 -> 109.0 mm
- net RST: track 48.9 -> 51.3 mm, vias 2 -> 1
- net BAT_P: track 16.3 -> 18.6 mm
- net layer_cluster_B: track 26.4 -> 24.2 mm
- net ring_top_B: track 24.1 -> 25.8 mm
- net RAW: track 79.8 -> 81.6 mm
- net space_cluster_B: track 26.1 -> 27.6 mm
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